File: KiCAD Files/PWMGenerator/PWMGenerator.kicad_sch (KiCad schematic)
At the start: 24 parts, among them J1 12V DC, U1 TL074

Commit message: Updated Schematic
Parts:
- removed C3: 100n, symbol Device:C_Small
- removed R8: 100k, symbol Device:R_Small
- added D4: 1N4004, symbol Device:D_Small
- added J2: LOAD, symbol Connector_Generic:Conn_01x02
- added Q1: IRLIZ44N, Package_TO_SOT_THT:TO-220F-3_Vertical, symbol Transistor_FET:IRLIZ44N
- renumbered C2 to C1, C5 to C2, C1 to C3, D3 to D2, D2 to D3, R5 to R1, R2 to R10, R9 to R11, R6 to R2, R10 to R3, R11 to R4, R1 to R5, R7 to R6, R12 to R7, R4 to R8, R3 to R9, RV2 to RV1, RV1 to RV2
Connections:
- net GND: now also Q1.3 (S)
- net VCC: now also D4.1 (K), J2.1 (Pin_1); no longer C2.1, C4.1, D1.1 (K), R1.1, R3.1, R7.1
- net PW_OUT: now reaches R11.2
- net PW_OUT: now also Q1.1 (G)
- net TRI_OUT: now reaches R10.2
- new net: D4.2 (A), J2.2 (Pin_2), Q1.2 (D)
- new net +12V: C2.1, C4.1, D1.1 (K), R1.1, R3.1, R7.1
Other:
- moved on the sheet: C1, C2, C3, C4, D1, D2, D3, J1, R1, R10, R11, R2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

Commit message: Updated PCB Layout
Parts:
- removed J2: LOAD, symbol Connector_Generic:Conn_01x02
- added J2: Conn_01x04, Connector_PinHeader_2.54mm:PinHeader_1x04_P2.54mm_Vertical, symbol Connector_Generic:Conn_01x04
- added unit 5 of U1
- C1, C4: footprint (none) -> Capacitor_SMD:C_0805_2012Metric_Pad1.18x1.45mm_HandSolder
- C2: renamed from C3; footprint (none) -> Capacitor_SMD:C_0805_2012Metric_Pad1.18x1.45mm_HandSolder
- C3: renamed from C2; footprint (none) -> Capacitor_THT:CP_Radial_D10.0mm_P5.00mm
- D1, D3: footprint (none) -> Diode_THT:D_DO-35_SOD27_P7.62mm_Horizontal
- D2: footprint (none) -> LED_SMD:LED_1206_3216Metric_Pad1.42x1.75mm_HandSolder
- D4: footprint (none) -> Diode_THT:D_DO-41_SOD81_P7.62mm_Horizontal
- J1: footprint (none) -> TerminalBlock:TerminalBlock_MaiXu_MX126-5.0-02P_1x02_P5.00mm
- R1, R10, R11, R2: footprint (none) -> Resistor_SMD:R_0805_2012Metric_Pad1.20x1.40mm_HandSolder
- R3: renamed from R5; footprint (none) -> Resistor_SMD:R_0805_2012Metric_Pad1.20x1.40mm_HandSolder
- R4: renamed from R8; footprint (none) -> Resistor_SMD:R_0805_2012Metric_Pad1.20x1.40mm_HandSolder
- R5: renamed from R9; footprint (none) -> Resistor_SMD:R_0805_2012Metric_Pad1.20x1.40mm_HandSolder
- R6: renamed from R7; footprint (none) -> Resistor_SMD:R_0805_2012Metric_Pad1.20x1.40mm_HandSolder
- R7: renamed from R3; footprint (none) -> Resistor_SMD:R_0805_2012Metric_Pad1.20x1.40mm_HandSolder
- R8: renamed from R4; footprint (none) -> Resistor_SMD:R_0805_2012Metric_Pad1.20x1.40mm_HandSolder
- R9: renamed from R6; footprint (none) -> Resistor_SMD:R_0805_2012Metric_Pad1.20x1.40mm_HandSolder
- RV1: renamed from RV2; footprint (none) -> Potentiometer_THT:Potentiometer_Piher_PC-16_Single_Horizontal
- RV2: renamed from RV1; footprint (none) -> Potentiometer_THT:Potentiometer_Piher_PC-16_Single_Horizontal
- U1: footprint (none) -> Package_SO:SOIC-14_3.9x8.7mm_P1.27mm
Connections:
- net +12V: now also U1.4 (V+)
- net GND: now also U1.11 (V-)
- net PW_OUT: now also J2.4 (Pin_4)
- net TRI_OUT: now also J2.3 (Pin_3)
- net VCC: now also J2.1 (Pin_1)
- net at D4.2 (A), Q1.2 (D): now also J2.2 (Pin_2)
Other:
- moved on the sheet: C1, C2, C3, C4, D1, D2, D3, D4, J1, Q1, R1, R10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
